File: TiLDE.sch (EAGLE design)
At the start: 79 parts, among them IC1 L78M05CDT-TR, J1 Digital, J2 Analog, J4 POWER, Q1 CSM-3X-CRYSTALCSM-3X, U1 ATMEGA32U4-AU, U2 MCP73831, X1 USB-MICROB, X2 53048-02

Commit message: change usb, fix silk screen, add ucl logo
Parts:
- removed X1: USB-MICROB, SparkFun-Connectors:USB-MICROB
- added U$2: UCL-LOGO, TiLDA:UCL-LOGO
- added USB1: MICRO-USB-ZX62-B-5PA, serial:MICRO-USB-ZX62-B-5PA
Connections:
- net GND: now also USB1.G, USB1.GND1, USB1.GND2, USB1.GND3, USB1.GND4, USB1.GND5, USB1.GND6; no longer X1.GND
- net N$13: now also USB1.V; no longer X1.VBUS
- net N$2: now also USB1.D-; no longer X1.D-
- net N$5: now also USB1.D+; no longer X1.D+
Changed lines of the file:
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@@
 <part name="JP2" library="SparkFun-Aesthetics" deviceset="FIDUCIAL" device="1X2.5"/>
 <part name="JP6" library="SparkFun-Aesthetics" deviceset="FIDUCIAL" device="1X2.5"/>
-<part name="X1" library="SparkFun-Connectors" deviceset="USB" device="-MICROB"/>
 <part name="GND10" library="SparkFun" deviceset="GND" device=""/>
 <part name="X2" library="con-molex" deviceset="53?-02" device="048"/>
+<part name="USB1" library="serial" deviceset="MICRO-USB" device="-ZX62-B-5PA"/>
+<part name="U$2" library="TiLDA" deviceset="UCL-LOGO" device=""/>
 </parts>
 <sheets>
@@
 <instance part="JP2" gate="G$1" x="360.68" y="27.94"/>
 <instance part="JP6" gate="G$1" x="350.52" y="27.94"/>
-<instance part="X1" gate="G$1" x="55.88" y="55.88" rot="MR180"/>
-<instance part="GND10" gate="1" x="48.26" y="60.96" rot="R180"/>
+<instance part="GND10" gate="1" x="45.72" y="43.18" rot="R270"/>
 <instance part="X2" gate="-1" x="373.38" y="251.46" rot="R90"/>
 <instance part="X2" gate="-2" x="375.92" y="251.46" rot="R90"/>
+<instance part="USB1" gate="G$1" x="60.96" y="48.26" rot="MR0"/>
+<instance part="U$2" gate="G$1" x="314.96" y="38.1"/>
 </instances>
 <busses>
@@
 <wire x1="43.18" y1="53.34" x2="43.18" y2="60.96" width="0.1524" layer="91"/>
 <pinref part="F2" gate="G$1" pin="1"/>
-<pinref part="X1" gate="G$1" pin="VBUS"/>
 <wire x1="50.8" y1="53.34" x2="53.34" y2="53.34" width="0.1524" layer="91"/>
+<pinref part="USB1" gate="G$1" pin="V"/>
+<wire x1="53.34" y1="53.34" x2="55.88" y2="53.34" width="0.1524" layer="91"/>
 </segment>
 </net>
@@
 <segment>
 <pinref part="GND10" gate="1" pin="GND"/>
-<wire x1="48.26" y1="58.42" x2="48.26" y2="55.88" width="0.1524" layer="91"/>
-<pinref part="X1" gate="G$1" pin="GND"/>
-<wire x1="48.26" y1="55.88" x2="53.34" y2="55.88" width="0.1524" layer="91"/>
+<wire x1="48.26" y1="43.18" x2="53.34" y2="43.18" width="0.1524" layer="91"/>
+<pinref part="USB1" gate="G$1" pin="G"/>
+<wire x1="53.34" y1="43.18" x2="55.88" y2="43.18" width="0.1524" layer="91"/>
+<pinref part="USB1" gate="G$1" pin="GND5"/>
+<pinref part="USB1" gate="G$1" pin="GND4"/>
+<wire x1="68.58" y1="35.56" x2="66.04" y2="35.56" width="0.1524" layer="91"/>
+<pinref part="USB1" gate="G$1" pin="GND3"/>
+<wire x1="63.5" y1="35.56" x2="66.04" y2="35.56" width="0.1524" layer="91"/>
+<pinref part="USB1" gate="G$1" pin="GND2"/>
+<wire x1="63.5" y1="35.56" x2="60.96" y2="35.56" width="0.1524" layer="91"/>
+<pinref part="USB1" gate="G$1" pin="GND1"/>
+<wire x1="60.96" y1="35.56" x2="58.42" y2="35.56" width="0.1524" layer="91"/>
+<pinref part="USB1" gate="G$1" pin="GND6"/>
+<wire x1="58.42" y1="35.56" x2="55.88" y2="35.56" width="0.1524" layer="91"/>
+<wire x1="55.88" y1="35.56" x2="53.34" y2="35.56" width="0.1524" layer="91"/>
+<wire x1="53.34" y1="35.56" x2="53.34" y2="43.18" width="0.1524" layer="91"/>
 </segment>
 </net>
@@
 <wire x1="38.1" y1="50.8" x2="50.8" y2="50.8" width="0.1524" layer="91"/>
 <pinref part="R5" gate="G$1" pin="2"/>
-<pinref part="X1" gate="G$1" pin="D-"/>
 <wire x1="50.8" y1="50.8" x2="53.34" y2="50.8" width="0.1524" layer="91"/>
+<pinref part="USB1" gate="G$1" pin="D-"/>
+<wire x1="53.34" y1="50.8" x2="55.88" y2="50.8" width="0.1524" layer="91"/>
 </segment>
 </net>
@@
 <wire x1="38.1" y1="48.26" x2="50.8" y2="48.26" width="0.1524" layer="91"/>
 <pinref part="R4" gate="G$1" pin="2"/>
-<pinref part="X1" gate="G$1" pin="D+"/>
 <wire x1="50.8" y1="48.26" x2="53.34" y2="48.26" width="0.1524" layer="91"/>
-</segment>
-</net>
+<pinref part="USB1" gate="G$1" pin="D+"/>
+<wire x1="53.34" y1="48.26" x2="55.88" y2="48.26" width="0.1524" layer="91"/>
+</segment>
+</net>

Commit message: fix wireless MO and MI, remove un needed reset cap
Parts:
- removed C2: 0.1uF, resistor:C-EUC0603K
Connections:
- removed net RST: C2.1
- net MISO: now also JP5.7; no longer JP5.6
- net MOSI: now also JP5.6; no longer JP5.7
- net RESET: no longer C2.2
Other:
- note removed: "UART"
Changed lines of the file:
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@@
 <part name="GND32" library="SparkFun" deviceset="GND" device=""/>
 <part name="GND4" library="SparkFun" deviceset="GND" device=""/>
-<part name="C2" library="resistor" deviceset="C-EU" device="C0603K" value="0.1uF"/>
 <part name="P+1" library="SparkFun" deviceset="VCC" device=""/>
 <part name="P+8" library="SparkFun" deviceset="VCC" device=""/>
@@
 <text x="193.04" y="45.72" size="3.81" layer="95" ratio="12">Analog Supply</text>
 <text x="251.46" y="45.72" size="3.81" layer="95" ratio="12">Status LEDs</text>
-<text x="360.68" y="68.58" size="3.81" layer="95" ratio="12">UART</text>
 <text x="355.6" y="193.04" size="3.81" layer="95" ratio="12">Breakouts</text>
 <text x="99.06" y="254" size="3.81" layer="95" ratio="12">ATMEGA 32U4</text>
@@
 <instance part="GND30" gate="1" x="342.9" y="231.14"/>
 <instance part="GND32" gate="1" x="325.12" y="231.14"/>
-<instance part="GND4" gate="1" x="40.64" y="139.7" rot="MR0"/>
-<instance part="C2" gate="G$1" x="165.1" y="20.32" rot="R90"/>
+<instance part="GND4" gate="1" x="40.64" y="137.16" rot="MR0"/>
 <instance part="P+1" gate="1" x="172.72" y="35.56"/>
 <instance part="P+8" gate="1" x="20.32" y="256.54"/>
@@
 <attribute name="VALUE" x="43.18" y="142.621" size="1.778" layer="96"/>
 </instance>
-<instance part="GND22" gate="1" x="25.4" y="139.7" rot="MR0"/>
+<instance part="GND22" gate="1" x="25.4" y="137.16" rot="MR0"/>
 <instance part="Q1" gate="G$1" x="33.02" y="149.86" smashed="yes">
 <attribute name="NAME" x="32.258" y="153.416" size="1.6764" layer="95" ratio="11"/>
@@
 <wire x1="172.72" y1="20.32" x2="180.34" y2="20.32" width="0.1524" layer="91"/>
 <junction x="172.72" y="20.32"/>
-<junction x="170.18" y="20.32"/>
 <label x="190.5" y="20.32" size="1.778" layer="95" rot="R180" xref="yes"/>
 <pinref part="R2" gate="G$1" pin="1"/>
 <pinref part="S2" gate="S" pin="4"/>
-<pinref part="C2" gate="G$1" pin="2"/>
 <pinref part="S2" gate="S" pin="3"/>
 </segment>
@@
 </segment>
 <segment>
-<pinref part="JP5" gate="A" pin="6"/>
-<wire x1="48.26" y1="104.14" x2="58.42" y2="104.14" width="0.1524" layer="91"/>
-</segment>
-<segment>
 <pinref part="U$1" gate="G$1" pin="PB3(MISO)"/>
 <wire x1="195.58" y1="177.8" x2="205.74" y2="177.8" width="0.1524" layer="91"/>
+</segment>
+<segment>
+<pinref part="JP5" gate="A" pin="7"/>
+<wire x1="40.64" y1="101.6" x2="30.48" y2="101.6" width="0.1524" layer="91"/>
 </segment>
 </net>
@@
 </segment>
 <segment>
-<pinref part="JP5" gate="A" pin="7"/>
-<wire x1="40.64" y1="101.6" x2="30.48" y2="101.6" width="0.1524" layer="91"/>
-</segment>
-<segment>
 <pinref part="U$1" gate="G$1" pin="PB2(MOSI)"/>
 <wire x1="195.58" y1="180.34" x2="205.74" y2="180.34" width="0.1524" layer="91"/>
+</segment>
+<segment>
+<pinref part="JP5" gate="A" pin="6"/>
+<wire x1="48.26" y1="104.14" x2="58.42" y2="104.14" width="0.1524" layer="91"/>
 </segment>
 </net>
@@
 </segment>
 </net>
-<net name="RST" class="0">
-<segment>
-<wire x1="162.56" y1="20.32" x2="157.48" y2="20.32" width="0.1524" layer="91"/>
-<label x="157.48" y="20.32" size="1.778" layer="95" rot="R180" xref="yes"/>
-<pinref part="C2" gate="G$1" pin="1"/>
-</segment>
-</net>
 <net name="VBUS" class="0">
 <segment>
@@
 <pinref part="C15" gate="G$1" pin="2"/>
 <pinref part="GND22" gate="1" pin="GND"/>
-<wire x1="25.4" y1="142.24" x2="25.4" y2="139.7" width="0.1524" layer="91"/>
 </segment>
 <segment>
 <pinref part="C16" gate="G$1" pin="2"/>
 <pinref part="GND4" gate="1" pin="GND"/>
-<wire x1="40.64" y1="142.24" x2="40.64" y2="139.7" width="0.1524" layer="91"/>
 </segment>
 <segment>
@@
 </sheet>
 </sheets>
-<errors>
-</errors>
 </schematic>
 </drawing>
